File: kaboard/kaboard.kicad_sch (KiCad schematic)
At the start: 70 parts, among them SW1 SW_PUSH, SW10 SW_PUSH, SW11 SW_PUSH, SW12 SW_PUSH, SW13 SW_PUSH, SW14 SW_PUSH, SW15 SW_PUSH, SW16 SW_PUSH, SW17 SW_PUSH, SW18 SW_PUSH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

Commit message: mechanical stuff
Other:
- note added: "Diode Matrix"
- note added: "Pin Shorts (To avoid DRC errors) only one mcu will be on each board"
- note added: "Power switch & battery"
- note removed: "Pin Shorts (To avoid DRC errors)"
- moved on the sheet: BT1, D1, D10, D11, D12, D13, D14, D15, D16, D17, D18, D2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
