File: kaboard/kaboard.kicad_pcb (KiCad board)
At the start: 2 copper layers, 111.3 x 90.4 mm, 76 parts, among them SW1 SW_PUSH, SW10 SW_PUSH, SW11 SW_PUSH, SW12 SW_PUSH, SW13 SW_PUSH, SW14 SW_PUSH, SW15 SW_PUSH, SW16 SW_PUSH, SW17 SW_PUSH, SW18 SW_PUSH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

Commit message: pcb updates
Routing:
- net GND: track 0.00 -> 33.2 mm, vias 1 -> 2
- net vbat: vias 0 -> 1
Other:
- outline, holes or cut-outs redrawn
